File: slider_test/slider_test.sch (KiCad schematic (older format))
At the start: 8 parts

Commit message: ./slider_test: converted to new board format + little tweaks.
Parts:
- C1, C2: value C -> 20nF
- R1, R2: value R -> 1k
Connections:
- wire segments 18 -> 19
Changed lines of the file:
@@
-EESchema Schematic File Version 2  date Wed 18 Jul 2012 07:44:56 PM CEST
+EESchema Schematic File Version 2
 LIBS:my_parts
 LIBS:power
@@
 LIBS:valves
 LIBS:slider_test-cache
-EELAYER 25  0
+EELAYER 24 0
 EELAYER END
 $Descr User 6000 4329
@@
 Sheet 1 1
 Title "capsense slider"
-Date "18 jul 2012"
+Date "02 Jun 2014"
 Rev "0.1"
 Comp "2012 - blog.spitzenpfeil.org"
@@
 F 0 "#PWR01" H 3150 1150 30  0001 C CNN
 F 1 "GND" H 3150 1080 30  0001 C CNN
+F 2 "" H 3150 1150 60  0001 C CNN
+F 3 "" H 3150 1150 60  0001 C CNN
 	1    3150 1150
 	1    0    0    -1
@@
 F 0 "CS2" V 3550 950 50  0000 C CNN
 F 1 "slider" V 3650 950 40  0000 C CNN
+F 2 "" H 3600 950 60  0001 C CNN
+F 3 "" H 3600 950 60  0001 C CNN
 	1    3600 950
 	1    0    0    1
@@
 P 1050 1100
 F 0 "C2" V 1100 1200 50  0000 L CNN
-F 1 "C" V 1100 1000 50  0000 L CNN
+F 1 "20nF" V 1100 850 50  0000 L CNN
+F 2 "" H 1050 1100 60  0001 C CNN
+F 3 "" H 1050 1100 60  0001 C CNN
 	1    1050 1100
 	0    -1   -1   0
@@
 P 1600 1100
 F 0 "R2" V 1680 1100 50  0000 C CNN
-F 1 "R" V 1600 1100 50  0000 C CNN
+F 1 "1k" V 1600 1100 50  0000 C CNN
+F 2 "" H 1600 1100 60  0001 C CNN
+F 3 "" H 1600 1100 60  0001 C CNN
 	1    1600 1100
 	0    -1   -1   0
@@
 F 0 "TP2" H 2250 1400 40  0000 C CNN
 F 1 "TST" H 2250 1350 30  0000 C CNN
+F 2 "" H 2250 1100 60  0001 C CNN
+F 3 "" H 2250 1100 60  0001 C CNN
 	1    2250 1100
 	1    0    0    -1
@@
 F 0 "CS1" V 3550 1500 50  0000 C CNN
 F 1 "slider" V 3650 1500 40  0000 C CNN
+F 2 "" H 3600 1500 60  0001 C CNN
+F 3 "" H 3600 1500 60  0001 C CNN
 	1    3600 1500
 	1    0    0    1
@@
 F 0 "TP1" H 2250 1950 40  0000 C CNN
 F 1 "TST" H 2250 1900 30  0000 C CNN
+F 2 "" H 2250 1650 60  0001 C CNN
+F 3 "" H 2250 1650 60  0001 C CNN
 	1    2250 1650
 	1    0    0    -1
@@
 F 0 "#PWR02" H 3150 1700 30  0001 C CNN
 F 1 "GND" H 3150 1630 30  0001 C CNN
+F 2 "" H 3150 1700 60  0001 C CNN
+F 3 "" H 3150 1700 60  0001 C CNN
 	1    3150 1700
 	1    0    0    -1
@@
 P 1600 1650
 F 0 "R1" V 1680 1650 50  0000 C CNN
-F 1 "R" V 1600 1650 50  0000 C CNN
+F 1 "1k" V 1600 1650 50  0000 C CNN
+F 2 "" H 1600 1650 60  0001 C CNN
+F 3 "" H 1600 1650 60  0001 C CNN
 	1    1600 1650
 	0    -1   -1   0
@@
 P 1050 1650
 F 0 "C1" V 1100 1750 50  0000 L CNN
-F 1 "C" V 1100 1550 50  0000 L CNN
+F 1 "20nF" V 1100 1400 50  0000 L CNN
+F 2 "" H 1050 1650 60  0001 C CNN
+F 3 "" H 1050 1650 60  0001 C CNN
 	1    1050 1650
 	0    -1   -1   0
 $EndComp
+$Comp
+L PWR_FLAG #FLG03
+U 1 1 538CE7E0
+P 4050 1200
+F 0 "#FLG03" H 4050 1295 30  0001 C CNN
+F 1 "PWR_FLAG" H 4050 1380 30  0000 C CNN
+F 2 "" H 4050 1200 60  0000 C CNN
+F 3 "" H 4050 1200 60  0000 C CNN
+	1    4050 1200
+	1    0    0    -1
+$EndComp
+$Comp
+L GND #PWR04
+U 1 1 538CE7F4
+P 4050 1300
+F 0 "#PWR04" H 4050 1300 30  0001 C CNN
+F 1 "GND" H 4050 1230 30  0001 C CNN
+F 2 "" H 4050 1300 60  0000 C CNN
+F 3 "" H 4050 1300 60  0000 C CNN
+	1    4050 1300
+	1    0    0    -1
+$EndComp
+Wire Wire Line
+	4050 1200 4050 1300
 $EndSCHEMATC
